File: hardware/kicad/radio-mic-usb-ptt.kicad_pcb (KiCad board)
At the start: 2 copper layers, 72 x 42 mm, 23 parts, among them J1 KMC RJ45 MIC, U1 Seeed XIAO RP2040, U2 MCP6002T-E/MS

Commit message: Added some rough placement, u can connect hte dots :D
Parts:
- removed H1, H2, H3, H4: MountingHole_3.2mm, MountingHole_3.2mm
- removed R11, R6, R8: 1k, R_0603_1608Metric
- removed R13: 100k, R_0603_1608Metric
- removed R5: 200k, R_0603_1608Metric
- removed R7: 10k, R_0603_1608Metric
- added C6: 10uF, Capacitor_SMD:C_0603_1608Metric, F.Cu at (194.9, 95.8)
- added C7: 1uF, Capacitor_SMD:C_0603_1608Metric, F.Cu at (194.9, 98.3)
- added C8: 1uF, Capacitor_SMD:C_0603_1608Metric, F.Cu at (194.9, 100.8)
- added C9: 1uF, Capacitor_SMD:C_0603_1608Metric, F.Cu at (194.9, 103.3)
- added D2: GREEN, Diode_SMD:D_0603_1608Metric, F.Cu at (177.2, 91.5)
- added F1: 500mA, Fuse:Fuse_0805_2012Metric, F.Cu at (193.2, 91.9)
- added J2: USB_C_Receptacle_USB2.0_16P, Connector_USB:USB_C_Receptacle_HRO_TYPE-C-31-M-12, F.Cu at (185.0, 87.5)
- added J3: Conn_ARM_SWD_TagConnect_TC2030-NL, Connector:Tag-Connect_TC2030-IDC-NL_2x03_P1.27mm_Vertical, B.Cu at (185.0, 94.8)
- added J4: Conn_01x04, Connector_PinHeader_2.54mm:PinHeader_1x04_P2.54mm_Vertical, F.Cu at (177.0, 104.0)
- added U3: USBLC6-2SC6, Package_TO_SOT_SMD:SOT-23-6, F.Cu at (185.0, 94.8)
- added U4: AP2127K-3.3, Package_TO_SOT_SMD:SOT-23-5, F.Cu at (193.8, 86.4)
- C1, C2: footprint C_0603_1608Metric -> Capacitor_SMD:C_0603_1608Metric
- C3: value 1nF -> 10uF; footprint C_0603_1608Metric -> Capacitor_SMD:C_0603_1608Metric
- C4, C5: value 100nF -> 1uF; footprint C_0603_1608Metric -> Capacitor_SMD:C_0603_1608Metric
- D1: value PTT_LED -> RED; footprint LED_0603_1608Metric -> Diode_SMD:D_0603_1608Metric
- J1: value KMC RJ45 MIC -> KMC-30/KMC-32 RJ45 MIC; footprint RJ45_Amphenol_RJHSE5380 -> Connector_RJ:RJ45_Amphenol_RJHSE5380
- R1: value 2.2k -> 100kR; footprint R_0603_1608Metric -> Resistor_SMD:R_0603_1608Metric
- R2: value 100k -> 200kR; footprint R_0603_1608Metric -> Resistor_SMD:R_0603_1608Metric
- R3: value 100k -> 1kR; footprint R_0603_1608Metric -> Resistor_SMD:R_0603_1608Metric
- R4: value 10k -> 1kR; footprint R_0603_1608Metric -> Resistor_SMD:R_0603_1608Metric
- U1: value Seeed XIAO RP2040 -> STM32L432KCUx; footprint XIAO-RP2040-SMD -> Package_DFN_QFN:QFN-32-1EP_5x5mm_P0.5mm_EP3.45x3.45mm
- U2: value MCP6002T-E/MS -> TLV9001IDCK; footprint MSOP-8_3x3mm_P0.65mm -> Package_TO_SOT_SMD:SOT-353_SC-70-5
- moved J1 200.6 mm to (181.4, 120.1)
- moved R1 188.9 mm to (194.9, 105.8)
- moved C4 188.9 mm to (190.9, 103.3)
- moved R4 187.1 mm to (198.9, 100.8)
- moved R2 181.4 mm to (198.9, 95.8)
- moved R3 181.2 mm to (198.9, 98.3)
- moved U2 175.6 mm to (183.3, 109.5)
- moved C1 175.1 mm to (190.9, 95.8)
- moved C3 173.8 mm to (190.9, 100.8)
- moved C5 173.8 mm to (190.9, 105.8)
- moved C2 170.4 mm to (190.9, 98.3)
- moved U1 160.8 mm to (185.0, 103.4), turned to 90 degrees
- moved D1 132.0 mm to (177.2, 88.9)
Connections:
- C1 pad 1: MIC_RAW -> +5V
- C1 pad 2: MIC_AC -> GND
- C2 pad 1: VREF -> +5V
- C3 pad 1: MIC_ADC -> /MIC_RAW
- C3 pad 2: GND -> Net-(U2-+)
- C4 pad 1: PTT_GPIO -> +3V3
- D1 pad 1: LED_A -> Net-(D1-K)
- D1 pad 2: GND -> Net-(D1-A)
- J1 pad 1: (no net) -> /UP_RAW
- J1 pad 2: (no net) -> +5V
- J1 pad 4: PTT_RAW -> /PTT_RAW
- J1 pad 6: MIC_RAW -> /MIC_RAW
- J1 pad 8: (no net) -> /DOWN_RAW
- J1 pad SH: GND -> (no net)
- R1 pad 1: +3V3 -> +5V
- R1 pad 2: MIC_RAW -> Net-(U2-+)
- R2 pad 1: +3V3 -> Net-(U2-+)
- R2 pad 2: VREF -> GND
- R3 pad 1: VREF -> Net-(D1-K)
- R4 pad 1: NINV -> Net-(D2-K)
- R4 pad 2: VREF -> GND
- U1 pad 1: MIC_ADC -> +3V3
- U1 pad 10: (no net) -> unconnected-(U1-PA4-Pad10)
- U1 pad 11: PTT_LED_DRIVE -> unconnected-(U1-PA5-Pad11)
- U1 pad 12: +3V3 -> unconnected-(U1-PA6-Pad12)
- U1 pad 13: GND -> unconnected-(U1-PA7-Pad13)
- U1 pad 14: (no net) -> /UP_RAW
- U1 pad 2: (no net) -> unconnected-(U1-PC14-Pad2)
- U1 pad 3: (no net) -> unconnected-(U1-PC15-Pad3)
- U1 pad 4: (no net) -> /~{RESET}
- U1 pad 5: (no net) -> +3V3
- U1 pad 6: (no net) -> /MIC_IN
- U1 pad 7: PTT_GPIO -> unconnected-(U1-PA1-Pad7)
- U1 pad 8: (no net) -> Net-(J4-Pin_2)
- U1 pad 9: (no net) -> Net-(J4-Pin_3)
- U2 pad 1: MIC_AMP -> Net-(U2-+)
- U2 pad 2: NINV -> GND
- U2 pad 3: MIC_AC -> /MIC_IN
- U2 pad 4: GND -> /MIC_IN
- U2 pad 5: VREF -> +5V
Routing:
- net GND: track 140.3 -> 0.00 mm, vias 2 -> 0
- net +3V3: track 79.8 -> 0.00 mm
- net PTT_RAW: track 34.5 -> 0.00 mm
- net PTT_GPIO: track 32.7 -> 0.00 mm
- net MIC_AMP: track 24.1 -> 0.00 mm
- net VREF: track 22.8 -> 0.00 mm
- net PTT_LED_DRIVE: track 19.2 -> 0.00 mm
- net MIC_RAW: track 18.8 -> 0.00 mm
- net MIC_AC: track 17.1 -> 0.00 mm
- net MIC_ADC: track 15.0 -> 0.00 mm
- net NINV: track 13.8 -> 0.00 mm
- net LED_A: track 2.40 -> 0.00 mm
Other:
- board size 72 x 42 mm -> 20 x 44 mm
- board text removed: "RJ45 MIC"
- board text removed: "USB-C ->"
- board text removed: "radio-mic-usb-ptt RevA"
