File: hardware/kicad/radio-mic-usb-ptt.kicad_sch (KiCad schematic)
At the start: 30 parts, among them J1 KMC-30/KMC-32 RJ45 MIC, U1 Seeed XIAO RP2040, U2 MCP6002T-E/MS

Commit message: reworked in 15 minutes btw
Parts:
- removed C1, C2: 1uF, radio-mic-usb-ptt:C_0603_1608Metric, symbol radio-mic-usb-ptt:C
- removed C3: 1nF, radio-mic-usb-ptt:C_0603_1608Metric, symbol radio-mic-usb-ptt:C
- removed C4, C5: 100nF, radio-mic-usb-ptt:C_0603_1608Metric, symbol radio-mic-usb-ptt:C
- removed D1: PTT_LED, radio-mic-usb-ptt:LED_0603_1608Metric, symbol radio-mic-usb-ptt:LED
- removed PF1, PF2: PWR_FLAG, symbol radio-mic-usb-ptt:PWR_FLAG
- removed R1: 2.2k, radio-mic-usb-ptt:R_0603_1608Metric, symbol radio-mic-usb-ptt:R
- removed R10, R4, R7, R9: 10k, radio-mic-usb-ptt:R_0603_1608Metric, symbol radio-mic-usb-ptt:R
- removed R11, R14, R15, R6, R8: 1k, radio-mic-usb-ptt:R_0603_1608Metric, symbol radio-mic-usb-ptt:R
- removed R12: DNP_0R_MIC_PWR, radio-mic-usb-ptt:R_0603_1608Metric, symbol radio-mic-usb-ptt:R
- removed R13, R2, R3: 100k, radio-mic-usb-ptt:R_0603_1608Metric, symbol radio-mic-usb-ptt:R
- removed R5: 200k, radio-mic-usb-ptt:R_0603_1608Metric, symbol radio-mic-usb-ptt:R
- removed TP1: MIC_RAW, radio-mic-usb-ptt:TestPoint_THTPad_D1.5mm, symbol radio-mic-usb-ptt:TestPoint
- removed TP2: MIC_ADC, radio-mic-usb-ptt:TestPoint_THTPad_D1.5mm, symbol radio-mic-usb-ptt:TestPoint
- removed TP3: PTT_GPIO, radio-mic-usb-ptt:TestPoint_THTPad_D1.5mm, symbol radio-mic-usb-ptt:TestPoint
- removed TP4: GND, radio-mic-usb-ptt:TestPoint_THTPad_D1.5mm, symbol radio-mic-usb-ptt:TestPoint
- removed U1: Seeed XIAO RP2040, Seeed_Studio_XIAO_Series:XIAO-RP2040-SMD, symbol radio-mic-usb-ptt:XIAO_RP2040_SMD
- removed U2: MCP6002T-E/MS, radio-mic-usb-ptt:MSOP-8_3x3mm_P0.65mm, symbol radio-mic-usb-ptt:MCP6002_MSOP8
- added C1, C2, C4, C5, C7, C8, C9: 1uF, symbol Device:C_Small
- added C3, C6: 10uF, symbol Device:C_Small
- added D1: RED, symbol Device:LED_Small
- added D2: GREEN, symbol Device:LED_Small
- added F1: 500mA, symbol Device:Polyfuse_Small
- added J2: USB_C_Receptacle_USB2.0_16P, symbol Connector:USB_C_Receptacle_USB2.0_16P
- added J3: Conn_ARM_SWD_TagConnect_TC2030-NL, Connector:Tag-Connect_TC2030-IDC-NL_2x03_P1.27mm_Vertical, symbol Connector:Conn_ARM_SWD_TagConnect_TC2030-NL
- added J4: Conn_01x04, symbol Connector_Generic:Conn_01x04
- added R1: 100kR, symbol Device:R_Small_US
- added R2: 200kR, symbol Device:R_Small_US
- added R3, R4: 1kR, symbol Device:R_Small_US
- added U1: STM32L432KCUx, Package_DFN_QFN:QFN-32-1EP_5x5mm_P0.5mm_EP3.45x3.45mm, symbol MCU_ST_STM32L4:STM32L432KCUx
- added U2: TLV9001IDCK, Package_TO_SOT_SMD:SOT-353_SC-70-5, symbol Amplifier_Operational:TLV9001IDCK
- added U3: USBLC6-2SC6, Package_TO_SOT_SMD:SOT-23-6, symbol Power_Protection:USBLC6-2SC6
- added U4: AP2127K-3.3, Package_TO_SOT_SMD:SOT-23-5, symbol Regulator_Linear:AP2127K-3.3
Connections:
- net +3V3: now also C4.1, C5.1, C6.2, C7.1, C9.1, J3.1 (VCC), J4.1 (Pin_1), U1.1 (VDD), U1.17 (VDD), U1.5 (VDDA), U4.5 (VOUT)
- net DOWN_RAW: now also U1.26 (PB3)
- net GND: now also C1.2, C2.2, C4.2, C5.2, C6.1, C7.2, C8.2, C9.2, J2.A1 (GND), J2.A12 (GND), J2.B1 (GND), J2.B12 (GND), J2.SH (SHIELD), J3.5 (GND), J4.4 (Pin_4), R2.2, R3.2, R4.2, U1.16 (VSS), U1.32 (VSS), U1.33 (VSS), U2.2 (V-), U3.2 (GND), U4.2 (GND)
- net MIC_RAW: now also C3.1
- net PTT_RAW: now also U1.15 (PB1)
- net UP_RAW: now also U1.14 (PB0)
- net MIC_PWR renamed +5V
- net +5V: now also C1.1, C2.1, C8.1, F1.2, R1.1, U2.5 (V+), U4.1 (VIN), U4.3 (EN)
- new net: F1.1, J2.A4 (VBUS), J2.A9 (VBUS), J2.B4 (VBUS), J2.B9 (VBUS), U3.5 (VBUS)
- new net: D1.1 (K), R3.1
- new net: D1.2 (A), U1.27 (PB4)
- new net: C3.2, R1.2, R2.1, U2.1 (+)
- new net: D2.1 (K), R4.1
- new net: D2.2 (A), U1.28 (PB5)
- new net: J4.2 (Pin_2), U1.8 (PA2)
- new net: J4.3 (Pin_3), U1.9 (PA3)
- new net BOOT0: U1.31 (PH3)
- new net CC1: J2.A5 (CC1)
- new net CC2: J2.B5 (CC2)
- new net D+: J2.A6 (D+), J2.B6 (D+), U1.22 (PA12), U3.3 (I/O2), U3.4 (I/O2)
- new net D-: J2.A7 (D-), J2.B7 (D-), U1.21 (PA11), U3.1 (I/O1), U3.6 (I/O1)
- new net MIC_IN: U1.6 (PA0), U2.3 (-), U2.4
- new net SWCLK: J3.4 (SWCLK), U1.24 (PA14)
- new net SWDIO: J3.2 (SWDIO), U1.23 (PA13)
- new net ~{RESET}: J3.3 (~{RESET}), U1.4 (NRST)
- no-connect marks 11 -> 16
Other:
- note added: "i2cjak wuz here"
- moved on the sheet: J1

Commit message: Added some rough placement, u can connect hte dots :D
Parts:
- C1, C2, C3, C4, C5, C6, C7, C8, C9: footprint (none) -> Capacitor_SMD:C_0603_1608Metric
- D1, D2: footprint (none) -> Diode_SMD:D_0603_1608Metric
- F1: footprint (none) -> Fuse:Fuse_0805_2012Metric
- J2: footprint (none) -> Connector_USB:USB_C_Receptacle_HRO_TYPE-C-31-M-12
- J4: footprint (none) -> Connector_PinHeader_2.54mm:PinHeader_1x04_P2.54mm_Vertical
- R1, R2, R3, R4: footprint (none) -> Resistor_SMD:R_0603_1608Metric
Changed lines of the file:
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@@
 			)
 		)
-		(property "Footprint" ""
+		(property "Footprint" "Fuse:Fuse_0805_2012Metric"
 			(at 109.22 52.07 0)
 			(hide yes)
@@
 			)
 		)
-		(property "Footprint" ""
+		(property "Footprint" "Diode_SMD:D_0603_1608Metric"
 			(at 158.75 110.49 90)
 			(hide yes)
@@
 			)
 		)
-		(property "Footprint" ""
+		(property "Footprint" "Resistor_SMD:R_0603_1608Metric"
 			(at 113.03 107.95 0)
 			(hide yes)
@@
 			)
 		)
-		(property "Footprint" ""
+		(property "Footprint" "Capacitor_SMD:C_0603_1608Metric"
 			(at 171.45 67.31 0)
 			(hide yes)
@@
 			)
 		)
-		(property "Footprint" ""
+		(property "Footprint" "Diode_SMD:D_0603_1608Metric"
 			(at 172.72 113.03 90)
 			(hide yes)
@@
 			)
 		)
-		(property "Footprint" ""
+		(property "Footprint" "Capacitor_SMD:C_0603_1608Metric"
 			(at 153.67 67.31 0)
 			(hide yes)
@@
 			)
 		)
-		(property "Footprint" ""
+		(property "Footprint" "Connector_USB:USB_C_Receptacle_HRO_TYPE-C-31-M-12"
 			(at 69.85 68.58 0)
 			(hide yes)
@@
 			)
 		)
-		(property "Footprint" ""
+		(property "Footprint" "Capacitor_SMD:C_0603_1608Metric"
 			(at 85.09 119.38 0)
 			(hide yes)
@@
 			)
 		)
-		(property "Footprint" ""
+		(property "Footprint" "Connector_PinHeader_2.54mm:PinHeader_1x04_P2.54mm_Vertical"
 			(at 223.52 87.63 0)
 			(hide yes)
@@
 			)
 		)
-		(property "Footprint" ""
+		(property "Footprint" "Resistor_SMD:R_0603_1608Metric"
 			(at 158.75 115.57 0)
 			(hide yes)
@@
 			)
 		)
-		(property "Footprint" ""
+		(property "Footprint" "Capacitor_SMD:C_0603_1608Metric"
 			(at 180.34 67.31 0)
 			(hide yes)
@@
 			)
 		)
-		(property "Footprint" ""
+		(property "Footprint" "Capacitor_SMD:C_0603_1608Metric"
 			(at 128.27 57.15 0)
 			(hide yes)
@@
 			)
 		)
-		(property "Footprint" ""
+		(property "Footprint" "Capacitor_SMD:C_0603_1608Metric"
 			(at 109.22 57.15 0)
 			(hide yes)
@@
 			)
 		)
-		(property "Footprint" ""
+		(property "Footprint" "Capacitor_SMD:C_0603_1608Metric"
 			(at 104.14 119.38 0)
 			(hide yes)
@@
 			)
 		)
-		(property "Footprint" ""
+		(property "Footprint" "Capacitor_SMD:C_0603_1608Metric"
 			(at 128.27 109.22 0)
 			(hide yes)
@@
 			)
 		)
-		(property "Footprint" ""
+		(property "Footprint" "Capacitor_SMD:C_0603_1608Metric"
 			(at 162.56 67.31 0)
 			(hide yes)
@@
 			)
 		)
-		(property "Footprint" ""
+		(property "Footprint" "Resistor_SMD:R_0603_1608Metric"
 			(at 172.72 118.11 0)
 			(hide yes)
@@
 			)
 		)
-		(property "Footprint" ""
+		(property "Footprint" "Resistor_SMD:R_0603_1608Metric"
 			(at 113.03 130.81 0)
 			(hide yes)
